File: Electrical Hardware/EAGLE Circuits/Low-Noise_Amp/Anti-Aliasing-Filter/AntiAlias Filter_Diff_Active.brd (EAGLE design)
At the start: 74.9 x 37.8 mm, 62 parts, among them U1 TLV272IS-13SO8_DIO-M, X1 BU-SMA-V, X2 BU-SMA-V, X3 BU-SMA-V, X4 BU-SMA-V

Commit message: Update sample holder+AA filter
Parts:
- removed D1, D2, D3, D4: (no value), diode:SMB
- added C19, C20: (no value), Favorite_Parts:C1206
- added IC1: 78L05F, linear:SOT89
- added U$1: 79LXX, VREG_L78L12ABUTR:VREG_L78L12ABUTR
- C1: value 3u -> 3n
- moved R13 4.58 mm to (27.9, 14.0), turned to 180 degrees
- moved C4 1.80 mm to (31.8, 16.5), flipped to the top
- moved C15 1.27 mm to (44.5, 15.2)
- moved C3 1.27 mm to (40.6, 16.5), flipped to the top
- moved R9 1.27 mm to (36.8, 10.2)
- turned R14 to 0 degrees
Connections:
- removed net N$5: D1.A, D3.C
- removed net N$6: D2.C, D4.A
- net +9V: now also C19.1, IC1.3; no longer D3.A
- net -9V: now also C20.1, U$1.2; no longer D4.C
- net GND: now also C19.2, C20.2, IC1.2, IC1.2@1, U$1.1
- net VS+: now also IC1.1; no longer D1.C
- net VS-: now also U$1.3; no longer D2.A
Routing:
- net +9V: track 15.8 -> 29.8 mm
- net -9V: track 30.4 -> 42.6 mm
- net VS-: track 37.8 -> 49.5 mm
- net GND: track 0.23 -> 10.9 mm, vias 26 -> 33
- net VS+: track 40.7 -> 48.1 mm
- net N$5: track 5.76 -> 0.00 mm
- net N$6: track 4.49 -> 0.00 mm
- net N$10: track 12.9 -> 15.4 mm
- net N$13: track 3.53 -> 2.26 mm
- net N$19: track 11.2 -> 12.4 mm
