File: Electrical Hardware/EAGLE Circuits/Low-Noise_Amp/Anti-Aliasing-Filter/AntiAlias Filter_Diff_Active.sch (EAGLE design)
At the start: 62 parts, among them U1 TLV272IS-13SO8_DIO-M, X1 BU-SMA-V, X2 BU-SMA-V, X3 BU-SMA-V, X4 BU-SMA-V

Commit message: Update sample holder+AA filter
Parts:
- removed D1, D2, D3, D4: (no value), diode:DIODE-SMB
- added C19, C20: (no value), Favorite_Parts:C-EUC1206
- added IC1: 78L05F, linear:78L05F
- added U$1: 79LXX, VREG_L78L12ABUTR:79LXX
- C1: value 3u -> 3n
Connections:
- removed net N$5: D1.A, D3.C
- removed net N$6: D2.C, D4.A
- net +9V: now also C19.1, IC1.VI; no longer D3.A
- net -9V: now also C20.1, U$1.P$2; no longer D4.C
- net GND: now also C19.2, C20.2, IC1.GND, IC1.GND@1, U$1.P$1
- net VS+: now also IC1.VO; no longer D1.C
- net VS-: now also U$1.P$3; no longer D2.A
Other:
- moved on the sheet: C4, C6, TP2
